File: KiCAD/avrComponentTester-Jose_Miquel_2-layer/avrComponentTester-Jose_Miquel_2-layer.kicad_pcb (KiCad board)
At the start: 2 copper layers, 11 parts, among them J4 3-pin_test_header, SW1 EC11, U1 ST7735_1.8

Commit message: New PCB and some READMEs
Parts:
- moved H4 25.4 mm to (95.2, 48.3)
- moved H2 7.73 mm to (95.2, 108.0)
- moved J4 1.27 mm to (186.7, 87.6)
- moved H1 1.27 mm to (186.7, 48.3)
- moved H3 1.27 mm to (186.7, 108.0)

Commit message: pcb
Parts:
- added Q1: 2N3904, My_Misc:TO-92_Inline_Wide_large, F.Cu at (106.0, 95.9)
- added Q2: 2N3904, My_Misc:TO-92_Inline_Wide_large, F.Cu at (150.5, 50.8)
- added Q3: 2N3906, My_Misc:TO-92_Inline_Wide_large, F.Cu at (108.0, 71.8)
- added U2: ATmega328P-PU, Package_DIP:DIP-28_W7.62mm_LongPads, F.Cu at (144.8, 86.4)
- added UC1: L78L05_TO92, My_Misc:TO-92_Inline_Wide_large, F.Cu at (99.7, 81.3)
- added UR1: TL431LP, My_Misc:TO-92_Inline_Wide_large, F.Cu at (148.0, 97.2)
- moved H1 100.8 mm to (101.6, 102.2)
- moved H2 94.8 mm to (189.9, 102.2)
- moved H3 58.5 mm to (189.9, 49.5)
- moved R21 46.4 mm to (177.8, 87.6)
- moved R22 36.5 mm to (173.4, 87.6), turned to 270 degrees
- moved C3 21.1 mm to (130.8, 68.6)
- moved J4 15.9 mm to (196.2, 74.9)
- moved C1 13.7 mm to (130.8, 72.4)
- moved SW1 9.20 mm to (176.5, 60.3)
- moved H4 6.48 mm to (101.6, 49.5)
