File: KiCAD/avrComponentTester/avrComponentTester.kicad_pcb (KiCad board)
At the start: 2 copper layers, 104.1 x 61.6 mm, 68 parts, among them J1 2-pin_power_input_header, J2 8-15VDC In, J3 3-pin_test_header, J4 3-pin_test_header, Q1 2N3904, Q2 2N3904, Q3 2N3906, SW1 RotaryEncoder_Switch, U1 ST7735_1.8"_TFT_128x160, U2 ATmega328P-PU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

Commit message: kicad, readme
Other:
- board text added: "${TITLE}-${REVISION} Design: Jon Sagebrand github.com/jonsag"
- board text removed: "avrComponentTester 0.5 Design: Jon Sagebrand github.com/jonsag"
Changed lines of the file:
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@@
   )
   (paper "A4")
+  (title_block
+    (title "avrComponentTester")
+    (date "2022-09-09")
+    (rev "0.5")
+  )
   (layers
     (0 "F.Cu" signal)
@@
     (effects (font (size 1 1) (thickness 0.15)))
   )
-  (gr_text "avrComponentTester 0.5\nDesign: Jon Sagebrand\ngithub.com/jonsag" (at 167.64 48.26) (layer "F.SilkS")
+  (gr_text "${TITLE}-${REVISION}\nDesign: Jon Sagebrand\ngithub.com/jonsag" (at 167.64 48.26) (layer "F.SilkS")
     (effects (font (size 1 1) (thickness 0.15)) (justify left))
   )
