File: KiCAD/avrComponentTester/avrComponentTester.kicad_sch (KiCad schematic)
At the start: 68 parts, among them J1 2-pin_power_input_header, J2 8-15VDC In, J3 3-pin_test_header, J4 3-pin_test_header, Q1 2N3904, Q2 2N3904, Q3 2N3906, SW1 RotaryEncoder_Switch, U1 ST7735_1.8"_TFT_128x160, U2 ATmega328P-PU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

Commit message: deletions and moving to new kicad dir
Parts:
- U2: footprint Package_DIP:DIP-28_W7.62mm -> My_Misc:DIP-28_W7.62mm_LongPads w socket
Changed lines of the file:
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@@
       (effects (font (size 1.27 1.27)) (justify right))
     )
-    (property "Footprint" "Package_DIP:DIP-28_W7.62mm" (id 2) (at 146.05 81.28 0)
+    (property "Footprint" "My_Misc:DIP-28_W7.62mm_LongPads w socket" (id 2) (at 146.05 81.28 0)
       (effects (font (size 1.27 1.27) italic) hide)
     )
@@
     )
     (path "/00000000-0000-0000-0000-00006027c604"
-      (reference "U2") (unit 1) (value "ATmega328P-PU") (footprint "Package_DIP:DIP-28_W7.62mm")
+      (reference "U2") (unit 1) (value "ATmega328P-PU") (footprint "My_Misc:DIP-28_W7.62mm_LongPads w socket")
     )
     (path "/00000000-0000-0000-0000-000060f0f960"

Commit message: kicad, readme
Other:
- title: (none) -> avrComponentTester
Changed lines of the file:
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@@
 (kicad_sch (version 20211123) (generator eeschema)
   (paper "A4")
+  (title_block
+    (title "avrComponentTester")
+    (date "2022-09-09")
+    (rev "0.5")
+  )
   (junction (at 107.95 168.91) (diameter 0) (color 0 0 0 0)
   )
